File: IMU.kicad_sch (KiCad schematic)
At the start: 13 parts, among them J11 BHI_JTAG_1V8, U10 TXB0106PW, U13 BHI260AP

Commit message: Routing done by @Turlinahi
Parts:
- U13: footprint hiro_samurai:XDCR_BHI260AP -> hiro_sumo:XDCR_BHI260AP
Changed lines of the file:
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@@
 			)
 		)
-		(property "Footprint" "hiro_samurai:XDCR_BHI260AP"
+		(property "Footprint" "hiro_sumo:XDCR_BHI260AP"
 			(at 211.455 102.87 0)
 			(effects
