File: hiro_samurai.kicad_pcb (KiCad board)
At the start: 4 copper layers, 103.5 x 65.5 mm, 159 parts, among them J1 BATTERY, J10 COLOR, J11 BHI_JTAG_1V8, J12 PMW, J13 LIFT, J14 KILL, J15 RGB_LED, J16 Debug_JTAG, J2 KILL, J3 CAN, J4 PNP1, J5 PNP2, J6 PWM1, J7 PWM2, J8 USB_C_Receptacle_USB2.0, J9 PNP_POWER, Q1 UMH3N, Q13 UMH3N, Q2 UMH3N, Q3 UMH3N, Q4 UMH3N, Q5 UMH3N, Q6 UMH3N, Q7 IRLML9303TRPBF, U1 STM32U585CITx, U10 TXB0106PW, U12 SPX3819M5-L-1-8, U13 BHI260AP, U14 TLP291, U15 TLP291, U2 ESD224DQA, U3 ESP32-S3-WROOM-2, U4 ESD224DQA, U5 TPS562212DRLR, U6 MIC5205-5.0YM5, U7 TJA1051T-3, U8 USBLC6-2SC6, U9 CP2105-F01-GM, Y1 16 Mhz

Commit message: Routing done by @Turlinahi
Parts:
- added kibuzzard-66A55516: G***, kibuzzard-66A55516, B.Cu at (130.2, 61.9)
- added kibuzzard-66A557E3: G***, kibuzzard-66A557E3, F.Cu at (84.0, 61.9)
- added kibuzzard-66A55816: G***, kibuzzard-66A55816, B.Cu at (157.2, 66.9)
- added kibuzzard-66A55828: G***, kibuzzard-66A55828, B.Cu at (156.9, 98.3)
- added kibuzzard-66A5583A: G***, kibuzzard-66A5583A, B.Cu at (107.3, 104.9)
- added kibuzzard-66A5585D: G***, kibuzzard-66A5585D, B.Cu at (89.9, 105.0)
- added kibuzzard-66A55877: G***, kibuzzard-66A55877, B.Cu at (75.9, 105.0)
- added kibuzzard-66A5588A: G***, kibuzzard-66A5588A, B.Cu at (77.0, 58.5)
- added kibuzzard-66A55897: G***, kibuzzard-66A55897, B.Cu at (88.0, 58.5)
- added kibuzzard-66A558AF: G***, kibuzzard-66A558AF, B.Cu at (103.7, 58.5)
- added kibuzzard-66A558D5: G***, kibuzzard-66A558D5, B.Cu at (99.3, 63.8)
- added kibuzzard-66A68797: G***, kibuzzard-66A68797, F.Cu at (152.9, 70.2)
- R8, R9: moved to B.Cu
- U13: footprint hiro_samurai:XDCR_BHI260AP -> hiro_sumo:XDCR_BHI260AP
- moved TP2 85.7 mm to (148.3, 102.6), turned to 90 degrees
- moved TP1 81.3 mm to (143.3, 104.1), turned to 90 degrees
- moved R9 51.9 mm to (114.9, 68.7), turned to 180 degrees
- moved R8 51.9 mm to (115.0, 67.0), turned to 180 degrees
- moved R7 38.1 mm to (114.9, 70.8)
- moved C13 3.60 mm to (119.1, 77.8), turned to 90 degrees
- moved H2 3.00 mm to (68.5, 61.4)
- moved H3 3.00 mm to (68.5, 103.4)
- moved C3 1.97 mm to (101.6, 107.7)
- moved C50 1.92 mm to (81.8, 107.7)
- moved C60 1.74 mm to (83.3, 109.2)
- moved Q6 1.34 mm to (67.6, 70.8)
- moved RN8 1.34 mm to (67.7, 73.8)
- moved RN9 1.34 mm to (67.6, 67.8)
- moved J4 1.24 mm to (67.0, 112.8)
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Routing:
- net +3V3: track 72.2 -> 342.3 mm, vias 6 -> 19
- net ~{STM_NRST}: track 2.02 -> 90.1 mm, vias 0 -> 10
- net GND: track 7.38 -> 76.5 mm, vias 2 -> 212
- net RGB_LED: track 0.00 -> 67.1 mm, vias 0 -> 2
- net VBAT: track 70.1 -> 136.5 mm, vias 4 -> 13
- net +5V: track 2.04 -> 66.4 mm, vias 0 -> 2
- net LIFT3: track 0.00 -> 50.8 mm, vias 0 -> 1
- net +1V8: track 27.2 -> 76.6 mm, vias 0 -> 11
- net Net-(R59-Pad1): track 0.00 -> 49.0 mm, vias 0 -> 4
- net COL2: track 0.00 -> 47.5 mm, vias 0 -> 1
- net LIFT2: track 0.00 -> 47.0 mm, vias 0 -> 3
- net LIFT1: track 0.00 -> 46.8 mm, vias 0 -> 1
- net Net-(R5-Pad2): track 0.00 -> 46.4 mm, vias 0 -> 6
- net LIFT4: track 0.00 -> 46.0 mm, vias 0 -> 2
- net COL1: track 0.00 -> 44.9 mm, vias 0 -> 3
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- removed copper zone on B.Cu, net GND
- removed copper zone on F.Cu, net GND
Other:
- board size 103.5 x 65.5 mm -> 99.6 x 64.2 mm
- board text added: "Ps 111:2"
